Commit message: 更换了smac和mppi算法

File: src/navigation/robot_navigation2/urdf/diff_drive_robot.urdf (robot description, URDF)
Before this commit: robot diff_drive_robot, 6 links, 5 joints
Joints:
- joint laser_joint: origin xyz=0.10 0 0.18 rpy=0 0 0 -> xyz=0.10 0.01 0.20 rpy=0 0 0

Commit message: 1

File: src/navigation/robot_navigation2/urdf/diff_drive_robot.urdf (robot description, URDF)
Before this commit: robot diff_drive_robot, 6 links, 5 joints
Joints:
- removed joint livox_joint
- added joint livox_to_laser_joint: type fixed, parent laser_link, child livox_frame, origin xyz=0 0 0 rpy=0 0 0

Commit message: 2026.2.5

File: src/navigation/robot_navigation2/urdf/diff_drive_robot.urdf (robot description, URDF)
Before this commit: robot diff_drive_robot, 6 links, 5 joints
Links:
- link base_link: geometry visual cylinder length=0.25 radius=0.251
Joints:
- joint base_footprint_joint: origin xyz=0 0 0.06 rpy=0 0 0 -> xyz=0 0 0.05 rpy=0 0 0
- joint laser_joint: origin xyz=0.10 0.01 0.20 rpy=0 0 0 -> xyz=0.22 0 0.25 rpy=0 0 0
- joint left_wheel_joint: origin xyz=0 0.15 -0.05 rpy=0 0 0 -> xyz=0 0.251 -0.075 rpy=0 0 0
- joint right_wheel_joint: origin xyz=0 -0.15 -0.05 rpy=0 0 0 -> xyz=0 -0.251 -0.075 rpy=0 0 0
